Commit message: ei isoja muutoksia

File: install/multi_robot_slam/share/multi_robot_slam/urdf/robot.urdf.xacro (robot description, xacro)
@@ -1 +1 @@
-/home/aisl/Documents/multi_robot_slam_ws/src/multi_robot_slam/urdf/robot.urdf.xacro
+/home/essivekkeli/multi_robot_slam_ws/src/multi_robot_slam/urdf/robot.urdf.xacro

File: src/multi_robot_slam/urdf/robot.urdf.xacro (robot description, xacro)
@@ -1,5 +1,5 @@
 <?xml version="1.0"?>
 <robot name="simple_robot" xmlns:xacro="http://www.ros.org/wiki/xacro">
-  <!-- Pass robot name from launch file -->
+  <!-- Robot namespace -->
   <xacro:arg name="robot_name" default="robot"/>
   <!-- Constants -->
@@ -9,7 +9,6 @@
   <xacro:property name="wheel_width" value="0.04"/>
   <xacro:property name="wheel_separation" value="0.3"/>
-  <!-- Base footprint (usually used as odom child frame) -->
+  <!-- ================= BASE ================= -->
   <link name="base_footprint"/>
-  <!-- Base link -->
   <link name="base_link">
     <visual>
@@ -28,5 +27,7 @@
     <inertial>
       <mass value="5.0"/>
-      <inertia ixx="0.01" ixy="0.0" ixz="0.0" iyy="0.01" iyz="0.0" izz="0.01"/>
+      <inertia ixx="0.01" ixy="0.0" ixz="0.0"
+               iyy="0.01" iyz="0.0"
+               izz="0.01"/>
     </inertial>
   </link>
@@ -36,6 +37,10 @@
     <origin xyz="0 0 0.05" rpy="0 0 0"/>
   </joint>
-  <!-- Lidar Link -->
-  <link name="lidar_link">
+  <!-- ================= LIDAR (FIXED) ================= -->
+  <!-- IMPORTANT:
+       Link name is now "lidar" (not lidar_link)
+       This MUST match the LaserScan frame_id
+  -->
+  <link name="lidar">
     <visual>
       <geometry>
@@ -53,15 +58,16 @@
     <inertial>
       <mass value="0.1"/>
-      <inertia ixx="0.0001" ixy="0.0" ixz="0.0" iyy="0.0001" iyz="0.0" izz="0.0001"/>
+      <inertia ixx="0.0001" ixy="0.0" ixz="0.0"
+               iyy="0.0001" iyz="0.0"
+               izz="0.0001"/>
     </inertial>
   </link>
   <joint name="lidar_joint" type="fixed">
     <parent link="base_link"/>
-    <child link="lidar_link"/>
+    <child link="lidar"/>
     <origin xyz="0 0 0.08" rpy="0 0 0"/>
   </joint>
-  <!-- ================== GAZEBO PLUGINS ================== -->
-  <!-- Lidar sensor (gpu_lidar) - publishes raw LaserScan data -->
-  <gazebo reference="lidar_link">
+  <!-- ================= GAZEBO LIDAR ================= -->
+  <gazebo reference="lidar">
     <sensor name="lidar" type="gpu_lidar">
       <pose>0 0 0 0 0 0</pose>
@@ -87,7 +93,8 @@
     </sensor>
   </gazebo>
-  <!-- Differential Drive Plugin - controls wheels, publishes odom, accepts cmd_vel -->
+  <!-- ================= DIFF DRIVE (MULTI-ROBOT SAFE) ================= -->
   <gazebo>
-    <plugin filename="gz-sim-diff-drive-system" name="gz::sim::systems::DiffDrive">
+    <plugin filename="gz-sim-diff-drive-system"
+            name="gz::sim::systems::DiffDrive">
       <left_joint>left_wheel_joint</left_joint>
       <right_joint>right_wheel_joint</right_joint>
@@ -96,6 +103,7 @@
       <topic>$(arg robot_name)/cmd_vel</topic>
       <odom_topic>$(arg robot_name)/odom</odom_topic>
-      <odom_frame>odom</odom_frame>
-      <child_frame_id>base_footprint</child_frame_id>
+      <!-- CRITICAL FIX -->
+      <odom_frame>$(arg robot_name)/odom</odom_frame>
+      <child_frame_id>$(arg robot_name)/base_footprint</child_frame_id>
       <publish_odom_tf>true</publish_odom_tf>
       <publish_wheel_tf>false</publish_wheel_tf>
@@ -103,11 +111,12 @@
     </plugin>
   </gazebo>
-  <!-- Pose Publisher - publishes gz.msgs.Pose_V for TF bridge -->
+  <!-- ================= POSE PUBLISHER ================= -->
   <gazebo>
-    <plugin filename="gz-sim-pose-publisher-system" name="gz::sim::systems::PosePublisher">
+    <plugin filename="gz-sim-pose-publisher-system"
+            name="gz::sim::systems::PosePublisher">
       <topic>$(arg robot_name)/tf</topic>
     </plugin>
   </gazebo>
-  <!-- Left Wheel -->
+  <!-- ================= WHEELS ================= -->
   <link name="left_wheel">
     <visual>
@@ -115,5 +124,5 @@
         <cylinder radius="${wheel_radius}" length="${wheel_width}"/>
       </geometry>
-      <origin xyz="0 0 0" rpy="1.5708 0 0"/> <!-- ≈ π/2 -->
+      <origin xyz="0 0 0" rpy="1.5708 0 0"/>
       <material name="gray">
         <color rgba="0.5 0.5 0.5 1"/>
@@ -128,5 +137,7 @@
     <inertial>
       <mass value="0.5"/>
-      <inertia ixx="0.0001" ixy="0.0" ixz="0.0" iyy="0.0001" iyz="0.0" izz="0.0001"/>
+      <inertia ixx="0.0001" ixy="0.0" ixz="0.0"
+               iyy="0.0001" iyz="0.0"
+               izz="0.0001"/>
     </inertial>
   </link>
@@ -137,5 +148,4 @@
     <axis xyz="0 1 0"/>
   </joint>
-  <!-- Right Wheel -->
   <link name="right_wheel">
     <visual>
@@ -156,5 +166,7 @@
     <inertial>
       <mass value="0.5"/>
-      <inertia ixx="0.0001" ixy="0.0" ixz="0.0" iyy="0.0001" iyz="0.0" izz="0.0001"/>
+      <inertia ixx="0.0001" ixy="0.0" ixz="0.0"
+               iyy="0.0001" iyz="0.0"
+               izz="0.0001"/>
     </inertial>
   </link>

Commit message: Global map works, but the quality of map is not good

File: install/multi_robot_slam/share/multi_robot_slam/urdf/robot.urdf.xacro (robot description, xacro)
@@ -1 +1,191 @@
-/home/aisl/Documents/multi_robot_slam_ws/src/multi_robot_slam/urdf/robot.urdf.xacro
+<?xml version="1.0"?>
+<robot name="simple_robot" xmlns:xacro="http://www.ros.org/wiki/xacro">
+  <!-- Robot namespace -->
+  <xacro:arg name="robot_name" default="robot"/>
+  <!-- Constants -->
+  <xacro:property name="base_radius" value="0.15"/>
+  <xacro:property name="base_height" value="0.1"/>
+  <xacro:property name="wheel_radius" value="0.05"/>
+  <xacro:property name="wheel_width" value="0.04"/>
+  <xacro:property name="wheel_separation" value="0.3"/>
+  <!-- ================= BASE ================= -->
+  <link name="base_footprint"/>
+  <link name="base_link">
+    <visual>
+      <geometry>
+        <cylinder radius="${base_radius}" length="${base_height}"/>
+      </geometry>
+      <material name="blue">
+        <color rgba="0 0 0.8 1"/>
+      </material>
+    </visual>
+    <collision>
+      <geometry>
+        <cylinder radius="${base_radius}" length="${base_height}"/>
+      </geometry>
+    </collision>
+    <inertial>
+      <mass value="5.0"/>
+      <inertia ixx="0.01" ixy="0.0" ixz="0.0"
+               iyy="0.01" iyz="0.0"
+               izz="0.01"/>
+    </inertial>
+  </link>
+  <joint name="base_joint" type="fixed">
+    <parent link="base_footprint"/>
+    <child link="base_link"/>
+    <origin xyz="0 0 0.05" rpy="0 0 0"/>
+  </joint>
+  <!-- ================= LIDAR (FIXED) ================= -->
+  <!-- IMPORTANT:
+       Link name is now "lidar" (not lidar_link)
+       This MUST match the LaserScan frame_id
+  -->
+  <link name="lidar">
+    <visual>
+      <geometry>
+        <cylinder radius="0.05" length="0.04"/>
+      </geometry>
+      <material name="black">
+        <color rgba="0 0 0 1"/>
+      </material>
+    </visual>
+    <collision>
+      <geometry>
+        <cylinder radius="0.05" length="0.04"/>
+      </geometry>
+    </collision>
+    <inertial>
+      <mass value="0.1"/>
+      <inertia ixx="0.0001" ixy="0.0" ixz="0.0"
+               iyy="0.0001" iyz="0.0"
+               izz="0.0001"/>
+    </inertial>
+  </link>
+  <joint name="lidar_joint" type="fixed">
+    <parent link="base_link"/>
+    <child link="lidar"/>
+    <origin xyz="0 0 0.08" rpy="0 0 0"/>
+  </joint>
+  <!-- ================= GAZEBO LIDAR ================= -->
+  <gazebo reference="lidar">
+    <sensor name="lidar" type="gpu_lidar">
+      <pose>0 0 0 0 0 0</pose>
+      <frame_name>$(arg robot_name)/lidar</frame_name>
+      <topic>$(arg robot_name)/scan</topic>
+      <update_rate>10</update_rate>
+      <lidar>
+        <scan>
+          <horizontal>
+            <samples>360</samples>
+            <resolution>1.0</resolution>
+            <min_angle>-3.14159</min_angle>
+            <max_angle>3.14159</max_angle>
+          </horizontal>
+        </scan>
+        <range>
+          <min>0.12</min>
+          <max>10.0</max>
+          <resolution>0.01</resolution>
+        </range>
+      </lidar>
+      <always_on>true</always_on>
+      <visualize>true</visualize>
+    </sensor>
+  </gazebo>
+  <!-- ================= DIFF DRIVE (MULTI-ROBOT SAFE) ================= -->
+  <gazebo>
+    <plugin filename="gz-sim-diff-drive-system"
+            name="gz::sim::systems::DiffDrive">
+      <left_joint>left_wheel_joint</left_joint>
+      <right_joint>right_wheel_joint</right_joint>
+      <wheel_separation>${wheel_separation}</wheel_separation>
+      <wheel_radius>${wheel_radius}</wheel_radius>
+      <topic>$(arg robot_name)/cmd_vel</topic>
+      <odom_topic>$(arg robot_name)/odom</odom_topic>
+      <!-- CRITICAL FIX -->
+      <odom_frame>$(arg robot_name)/odom</odom_frame>
+      <child_frame_id>$(arg robot_name)/base_footprint</child_frame_id>
+      <publish_odom>true</publish_odom>
+      <publish_odom_tf>true</publish_odom_tf>
+      <use_sim_time>true</use_sim_time>
+      <publish_wheel_tf>false</publish_wheel_tf>
+      <odom_publish_frequency>50</odom_publish_frequency>
+    </plugin>
+  </gazebo>
+  <!-- ================= POSE PUBLISHER ================= -->
+  <gazebo>
+    <plugin filename="gz-sim-pose-publisher-system"
+            name="gz::sim::systems::PosePublisher">
+      <topic>$(arg robot_name)/tf</topic>
+    </plugin>
+  </gazebo>
+  <gazebo>
+    <plugin filename="gz-sim-odometry-publisher-system"
+            name="gz::sim::systems::OdometryPublisher">
+      <odom_topic>$(arg robot_name)/odom</odom_topic>
+      <odom_frame>$(arg robot_name)/odom</odom_frame>
+      <robot_base_frame>$(arg robot_name)/base_footprint</robot_base_frame>
+      <odom_publish_frequency>50</odom_publish_frequency>
+    </plugin>
+  </gazebo>
+  <!-- ================= WHEELS ================= -->
+  <link name="left_wheel">
+    <visual>
+      <geometry>
+        <cylinder radius="${wheel_radius}" length="${wheel_width}"/>
+      </geometry>
+      <origin xyz="0 0 0" rpy="1.5708 0 0"/>
+      <material name="gray">
+        <color rgba="0.5 0.5 0.5 1"/>
+      </material>
+    </visual>
+    <collision>
+      <geometry>
+        <cylinder radius="${wheel_radius}" length="${wheel_width}"/>
+      </geometry>
+      <origin xyz="0 0 0" rpy="1.5708 0 0"/>
+    </collision>
+    <inertial>
+      <mass value="0.5"/>
+      <inertia ixx="0.0001" ixy="0.0" ixz="0.0"
+               iyy="0.0001" iyz="0.0"
+               izz="0.0001"/>
+    </inertial>
+  </link>
+  <joint name="left_wheel_joint" type="continuous">
+    <parent link="base_link"/>
+    <child link="left_wheel"/>
+    <origin xyz="0 ${wheel_separation/2} -0.03" rpy="0 0 0"/>
+    <axis xyz="0 1 0"/>
+  </joint>
+  <link name="right_wheel">
+    <visual>
+      <geometry>
+        <cylinder radius="${wheel_radius}" length="${wheel_width}"/>
+      </geometry>
+      <origin xyz="0 0 0" rpy="1.5708 0 0"/>
+      <material name="gray">
+        <color rgba="0.5 0.5 0.5 1"/>
+      </material>
+    </visual>
+    <collision>
+      <geometry>
+        <cylinder radius="${wheel_radius}" length="${wheel_width}"/>
+      </geometry>
+      <origin xyz="0 0 0" rpy="1.5708 0 0"/>
+    </collision>
+    <inertial>
+      <mass value="0.5"/>
+      <inertia ixx="0.0001" ixy="0.0" ixz="0.0"
+               iyy="0.0001" iyz="0.0"
+               izz="0.0001"/>
+    </inertial>
+  </link>
+  <joint name="right_wheel_joint" type="continuous">
+    <parent link="base_link"/>
+    <child link="right_wheel"/>
+    <origin xyz="0 ${-wheel_separation/2} -0.03" rpy="0 0 0"/>
+    <axis xyz="0 1 0"/>
+  </joint>
+</robot>

Commit message: save for the day

File: install/multi_robot_slam/share/multi_robot_slam/urdf/robot.urdf.xacro (robot description, xacro)
@@ -1,182 +1 @@
-<?xml version="1.0"?>
-<robot name="simple_robot" xmlns:xacro="http://www.ros.org/wiki/xacro">
-  <!-- Robot namespace -->
-  <xacro:arg name="robot_name" default="robot"/>
-  <!-- Constants -->
-  <xacro:property name="base_radius" value="0.15"/>
-  <xacro:property name="base_height" value="0.1"/>
-  <xacro:property name="wheel_radius" value="0.05"/>
-  <xacro:property name="wheel_width" value="0.04"/>
-  <xacro:property name="wheel_separation" value="0.3"/>
-  <!-- ================= BASE ================= -->
-  <link name="base_footprint"/>
-  <link name="base_link">
-    <visual>
-      <geometry>
-        <cylinder radius="${base_radius}" length="${base_height}"/>
-      </geometry>
-      <material name="blue">
-        <color rgba="0 0 0.8 1"/>
-      </material>
-    </visual>
-    <collision>
-      <geometry>
-        <cylinder radius="${base_radius}" length="${base_height}"/>
-      </geometry>
-    </collision>
-    <inertial>
-      <mass value="5.0"/>
-      <inertia ixx="0.01" ixy="0.0" ixz="0.0"
-               iyy="0.01" iyz="0.0"
-               izz="0.01"/>
-    </inertial>
-  </link>
-  <joint name="base_joint" type="fixed">
-    <parent link="base_footprint"/>
-    <child link="base_link"/>
-    <origin xyz="0 0 0.05" rpy="0 0 0"/>
-  </joint>
-  <!-- ================= LIDAR (FIXED) ================= -->
-  <!-- IMPORTANT:
-       Link name is now "lidar" (not lidar_link)
-       This MUST match the LaserScan frame_id
-  -->
-  <link name="lidar">
-    <visual>
-      <geometry>
-        <cylinder radius="0.05" length="0.04"/>
-      </geometry>
-      <material name="black">
-        <color rgba="0 0 0 1"/>
-      </material>
-    </visual>
-    <collision>
-      <geometry>
-        <cylinder radius="0.05" length="0.04"/>
-      </geometry>
-    </collision>
-    <inertial>
-      <mass value="0.1"/>
-      <inertia ixx="0.0001" ixy="0.0" ixz="0.0"
-               iyy="0.0001" iyz="0.0"
-               izz="0.0001"/>
-    </inertial>
-  </link>
-  <joint name="lidar_joint" type="fixed">
-    <parent link="base_link"/>
-    <child link="lidar"/>
-    <origin xyz="0 0 0.08" rpy="0 0 0"/>
-  </joint>
-  <!-- ================= GAZEBO LIDAR ================= -->
-  <gazebo reference="lidar">
-    <sensor name="lidar" type="gpu_lidar">
-      <pose>0 0 0 0 0 0</pose>
-      <frame_name>$(arg robot_name)/lidar</frame_name>
-      <topic>$(arg robot_name)/scan</topic>
-      <update_rate>10</update_rate>
-      <lidar>
-        <scan>
-          <horizontal>
-            <samples>360</samples>
-            <resolution>1.0</resolution>
-            <min_angle>-3.14159</min_angle>
-            <max_angle>3.14159</max_angle>
-          </horizontal>
-        </scan>
-        <range>
-          <min>0.12</min>
-          <max>10.0</max>
-          <resolution>0.01</resolution>
-        </range>
-      </lidar>
-      <always_on>true</always_on>
-      <visualize>true</visualize>
-    </sensor>
-  </gazebo>
-  <!-- ================= DIFF DRIVE (MULTI-ROBOT SAFE) ================= -->
-  <gazebo>
-    <plugin filename="gz-sim-diff-drive-system"
-            name="gz::sim::systems::DiffDrive">
-      <left_joint>left_wheel_joint</left_joint>
-      <right_joint>right_wheel_joint</right_joint>
-      <wheel_separation>${wheel_separation}</wheel_separation>
-      <wheel_radius>${wheel_radius}</wheel_radius>
-      <topic>$(arg robot_name)/cmd_vel</topic>
-      <odom_topic>$(arg robot_name)/odom</odom_topic>
-      <!-- CRITICAL FIX -->
-      <odom_frame>$(arg robot_name)/odom</odom_frame>
-      <child_frame_id>$(arg robot_name)/base_footprint</child_frame_id>
-      <publish_odom>true</publish_odom>
-      <publish_odom_tf>false</publish_odom_tf>
-      <use_sim_time>true</use_sim_time>
-      <publish_wheel_tf>false</publish_wheel_tf>
-      <odom_publish_frequency>50</odom_publish_frequency>
-    </plugin>
-  </gazebo>
-  <!-- ================= POSE PUBLISHER ================= -->
-  <gazebo>
-    <plugin filename="gz-sim-pose-publisher-system"
-            name="gz::sim::systems::PosePublisher">
-      <topic>$(arg robot_name)/tf</topic>
-    </plugin>
-  </gazebo>
-  <!-- ================= WHEELS ================= -->
-  <link name="left_wheel">
-    <visual>
-      <geometry>
-        <cylinder radius="${wheel_radius}" length="${wheel_width}"/>
-      </geometry>
-      <origin xyz="0 0 0" rpy="1.5708 0 0"/>
-      <material name="gray">
-        <color rgba="0.5 0.5 0.5 1"/>
-      </material>
-    </visual>
-    <collision>
-      <geometry>
-        <cylinder radius="${wheel_radius}" length="${wheel_width}"/>
-      </geometry>
-      <origin xyz="0 0 0" rpy="1.5708 0 0"/>
-    </collision>
-    <inertial>
-      <mass value="0.5"/>
-      <inertia ixx="0.0001" ixy="0.0" ixz="0.0"
-               iyy="0.0001" iyz="0.0"
-               izz="0.0001"/>
-    </inertial>
-  </link>
-  <joint name="left_wheel_joint" type="continuous">
-    <parent link="base_link"/>
-    <child link="left_wheel"/>
-    <origin xyz="0 ${wheel_separation/2} -0.03" rpy="0 0 0"/>
-    <axis xyz="0 1 0"/>
-  </joint>
-  <link name="right_wheel">
-    <visual>
-      <geometry>
-        <cylinder radius="${wheel_radius}" length="${wheel_width}"/>
-      </geometry>
-      <origin xyz="0 0 0" rpy="1.5708 0 0"/>
-      <material name="gray">
-        <color rgba="0.5 0.5 0.5 1"/>
-      </material>
-    </visual>
-    <collision>
-      <geometry>
-        <cylinder radius="${wheel_radius}" length="${wheel_width}"/>
-      </geometry>
-      <origin xyz="0 0 0" rpy="1.5708 0 0"/>
-    </collision>
-    <inertial>
-      <mass value="0.5"/>
-      <inertia ixx="0.0001" ixy="0.0" ixz="0.0"
-               iyy="0.0001" iyz="0.0"
-               izz="0.0001"/>
-    </inertial>
-  </link>
-  <joint name="right_wheel_joint" type="continuous">
-    <parent link="base_link"/>
-    <child link="right_wheel"/>
-    <origin xyz="0 ${-wheel_separation/2} -0.03" rpy="0 0 0"/>
-    <axis xyz="0 1 0"/>
-  </joint>
-</robot>
+/home/aisl/Documents/multi_robot_slam_ws/src/multi_robot_slam/urdf/robot.urdf.xacro
