Commit message: fixes

File: src/multi_robot_slam/urdf/robot.urdf.xacro (robot description, xacro)
@@ -1,4 +1,6 @@
 <?xml version="1.0"?>
 <robot name="simple_robot" xmlns:xacro="http://www.ros.org/wiki/xacro">
+  <!-- Pass robot name from launch file -->
+  <xacro:arg name="robot_name" default="robot"/>
   <!-- Constants -->
   <xacro:property name="base_radius" value="0.15"/>
@@ -7,6 +9,7 @@
   <xacro:property name="wheel_width" value="0.04"/>
   <xacro:property name="wheel_separation" value="0.3"/>
-  <!-- Base Link -->
+  <!-- Base footprint (usually used as odom child frame) -->
   <link name="base_footprint"/>
+  <!-- Base link -->
   <link name="base_link">
     <visual>
@@ -58,8 +61,10 @@
     <origin xyz="0 0 0.08" rpy="0 0 0"/>
   </joint>
-  <!-- Gazebo plugins and sensors -->
+  <!-- ================== GAZEBO PLUGINS ================== -->
+  <!-- Lidar sensor (gpu_lidar) - publishes raw LaserScan data -->
   <gazebo reference="lidar_link">
     <sensor name="lidar" type="gpu_lidar">
-      <topic>scan</topic>
+      <pose>0 0 0 0 0 0</pose>
+      <topic>$(arg robot_name)/scan</topic>
       <update_rate>10</update_rate>
       <lidar>
@@ -78,9 +83,9 @@
         </range>
       </lidar>
-      <always_on>1</always_on>
+      <always_on>true</always_on>
       <visualize>true</visualize>
     </sensor>
   </gazebo>
-  <!-- Differential drive plugin -->
+  <!-- Differential Drive Plugin - controls wheels, publishes odom, accepts cmd_vel -->
   <gazebo>
     <plugin filename="gz-sim-diff-drive-system" name="gz::sim::systems::DiffDrive">
@@ -89,9 +94,17 @@
       <wheel_separation>${wheel_separation}</wheel_separation>
       <wheel_radius>${wheel_radius}</wheel_radius>
+      <topic>$(arg robot_name)/cmd_vel</topic>
+      <odom_topic>$(arg robot_name)/odom</odom_topic>
+      <odom_frame>odom</odom_frame>
+      <child_frame_id>base_footprint</child_frame_id>
+      <publish_odom_tf>true</publish_odom_tf>
+      <publish_wheel_tf>false</publish_wheel_tf>
       <odom_publish_frequency>50</odom_publish_frequency>
-      <topic>cmd_vel</topic>
-      <odom_topic>odom</odom_topic>
-      <frame_id>odom</frame_id>
-      <child_frame_id>base_footprint</child_frame_id>
+    </plugin>
+  </gazebo>
+  <!-- Pose Publisher - publishes gz.msgs.Pose_V for TF bridge -->
+  <gazebo>
+    <plugin filename="gz-sim-pose-publisher-system" name="gz::sim::systems::PosePublisher">
+      <topic>$(arg robot_name)/tf</topic>
     </plugin>
   </gazebo>
@@ -102,5 +115,5 @@
         <cylinder radius="${wheel_radius}" length="${wheel_width}"/>
       </geometry>
-      <origin xyz="0 0 0" rpy="1.5707 0 0"/>
+      <origin xyz="0 0 0" rpy="1.5708 0 0"/> <!-- ≈ π/2 -->
       <material name="gray">
         <color rgba="0.5 0.5 0.5 1"/>
@@ -111,5 +124,5 @@
         <cylinder radius="${wheel_radius}" length="${wheel_width}"/>
       </geometry>
-      <origin xyz="0 0 0" rpy="1.5707 0 0"/>
+      <origin xyz="0 0 0" rpy="1.5708 0 0"/>
     </collision>
     <inertial>
@@ -130,5 +143,5 @@
         <cylinder radius="${wheel_radius}" length="${wheel_width}"/>
       </geometry>
-      <origin xyz="0 0 0" rpy="1.5707 0 0"/>
+      <origin xyz="0 0 0" rpy="1.5708 0 0"/>
       <material name="gray">
         <color rgba="0.5 0.5 0.5 1"/>
@@ -139,5 +152,5 @@
         <cylinder radius="${wheel_radius}" length="${wheel_width}"/>
       </geometry>
-      <origin xyz="0 0 0" rpy="1.5707 0 0"/>
+      <origin xyz="0 0 0" rpy="1.5708 0 0"/>
     </collision>
     <inertial>

Commit message: [200~AAccumulated point cloud fusion working, clear room structure visible in RViz

File: src/multi_robot_slam/urdf/robot.urdf.xacro (robot description, xacro)
@@ -66,5 +66,5 @@
     <parent link="base_link"/>
     <child link="lidar"/>
-    <origin xyz="0 0 0.08" rpy="0 0 0"/>
+    <origin xyz="0 0 0.4" rpy="0 0 0"/>
   </joint>
   <!-- ================= GAZEBO LIDAR ================= -->
@@ -86,6 +86,6 @@
             <samples>16</samples>
             <resolution>1.0</resolution>
-            <min_angle>-0.26180</min_angle>
-            <max_angle>0.26180</max_angle>
+            <min_angle>-0.5236</min_angle>
+            <max_angle>0.5236</max_angle>
           </vertical>
         </scan>
@@ -98,4 +98,36 @@
       <always_on>true</always_on>
       <visualize>true</visualize>
+    </sensor>
+  </gazebo>
+  <!-- ================= IMU ================= -->
+  <link name="imu_link">
+    <visual>
+      <geometry><box size="0.01 0.01 0.01"/></geometry>
+    </visual>
+  </link>
+  <joint name="imu_joint" type="fixed">
+    <parent link="base_link"/>
+    <child link="imu_link"/>
+    <origin xyz="0 0 0.05" rpy="0 0 0"/>
+  </joint>
+  <gazebo reference="imu_link">
+    <sensor name="imu" type="imu">
+      <always_on>true</always_on>
+      <update_rate>100</update_rate>
+      <topic>$(arg robot_name)/imu</topic>
+      <frame_name>$(arg robot_name)/imu_link</frame_name>
+      <imu>
+        <angular_velocity>
+          <x><noise type="gaussian"><mean>0</mean><stddev>0.009</stddev></noise></x>
+          <y><noise type="gaussian"><mean>0</mean><stddev>0.009</stddev></noise></y>
+          <z><noise type="gaussian"><mean>0</mean><stddev>0.009</stddev></noise></z>
+        </angular_velocity>
+        <linear_acceleration>
+          <x><noise type="gaussian"><mean>0</mean><stddev>0.021</stddev></noise></x>
+          <y><noise type="gaussian"><mean>0</mean><stddev>0.021</stddev></noise></y>
+          <z><noise type="gaussian"><mean>0</mean><stddev>0.021</stddev></noise></z>
+        </linear_acceleration>
+      </imu>
+      <plugin filename="gz-sim-imu-system" name="gz::sim::systems::Imu"/>
     </sensor>
   </gazebo>
